File: RPI-CM4-Breakout.brd (EAGLE design)
At the start: 70 x 59 mm, 27 parts, among them IC1 MC74VHC1G14DFT1G, J1 P1-100, J2 P101-200, J3 47571-0001

Commit message: Removed misleading pull-down on GLOBAL_EN
Parts:
- removed R6: 10k, microbuilder:_0402MP
Connections:
- net GLOBAL_EN: no longer R6.2
- net GND: no longer R6.1
